File: table-zamboni.kicad_sch (KiCad schematic)
At the start: 5 parts, among them U1 ESP32-C6-MINI-1

Commit message: Adding root page of schematic using esp32-wroom-32e
Parts:
- removed ME1, ME2, ME3, ME4: ~, symbol 2_Motor_with_Encoder:Motor_with_Encoder
- removed U1: ESP32-C6-MINI-1, RF_Module:ESP32-C6-MINI-1, symbol RF_Module:ESP32-C6-MINI-1
Other:
- removed sheet motor driver circuit
- added sheet ESP32 (esp32.kicad_sch)
- added sheet Motors (drive_motors.kicad_sch)
- added sheet Navigation Sensors (navigation_sensors.kicad_sch)
- added sheet Power Management + USB (pwr_mgmt.kicad_sch)
- note added: "* NOTE: This board is for prototyping and includes a few extra components to simplify the software development process."
- note added: "+5V_Battery"
- note added: "+BATT"
- note added: "3.3V"
- note added: "5V"
- note added: "BLOCK DIAGRAM"
- note added: "GPIO-Left_Motor"
- note added: "GPIO-Right_Motor"
- note added: "GPIO-Servo"
- note added: "I2C"
- note added: "SPI"
- note added: "TABLE ZAMBONI DEVELOPMENT BOARD"
- note added: "UART"
- note added: "USB_DATA"
- note added: "V_BUS"
- company: (none) -> Table Zamboni
- title: Table Zamboni Drive Train -> Development Board for Prototype
