File: Main_PCB/tof_sensors.kicad_sch (KiCad schematic)
At the start: 17 parts, among them Q501 2N7002, Q502 2N7002, U501 LP5907MFX-2.8, U502 VL53L4CD, U503 VL53L4CD

Commit message: Adding most recent version of schematic. I have now decided to use NiMH batteries instead of Li-ion because they are safer and I don't want to start a fire.
Parts:
- renumbered C505 to C504, C504 to C505, Q502 to Q501, Q501 to Q502, R502 to R501, R504 to R502, R507 to R503, R503 to R504, R501 to R505, R505 to R506
Changed lines of the file:
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@@
 		(dnp no)
 		(fields_autoplaced yes)
-		(property "Reference" "#PWR0516"
+		(property "Reference" "#PWR0515"
 			(at 217.17 147.32 0)
 			(effects
@@
 			(project "table-zamboni"
 				(path "/6b8b7632-a6ae-4a95-9a82-5604ab03d2a7/e5c972da-9e3b-4905-a822-7ee0d7b899b3"
-					(reference "#PWR0516")
+					(reference "#PWR0515")
 					(unit 1)
 				)
@@
 		(dnp no)
 		(fields_autoplaced yes)
-		(property "Reference" "C504"
+		(property "Reference" "C505"
 			(at 254 45.7199 0)
 			(effects
@@
 			(project "table-zamboni"
 				(path "/6b8b7632-a6ae-4a95-9a82-5604ab03d2a7/e5c972da-9e3b-4905-a822-7ee0d7b899b3"
-					(reference "C504")
+					(reference "C505")
 					(unit 1)
 				)
@@
 		(dnp no)
 		(fields_autoplaced yes)
-		(property "Reference" "R503"
+		(property "Reference" "R504"
 			(at 175.26 110.4899 0)
 			(effects
@@
 			(project "table-zamboni"
 				(path "/6b8b7632-a6ae-4a95-9a82-5604ab03d2a7/e5c972da-9e3b-4905-a822-7ee0d7b899b3"
-					(reference "R503")
+					(reference "R504")
 					(unit 1)
 				)
@@
 		(dnp no)
 		(fields_autoplaced yes)
-		(property "Reference" "R502"
+		(property "Reference" "R501"
 			(at 67.31 92.7099 0)
 			(effects
@@
 			(project "table-zamboni"
 				(path "/6b8b7632-a6ae-4a95-9a82-5604ab03d2a7/e5c972da-9e3b-4905-a822-7ee0d7b899b3"
-					(reference "R502")
+					(reference "R501")
 					(unit 1)
 				)
@@
 		(dnp no)
 		(fields_autoplaced yes)
-		(property "Reference" "#PWR0512"
+		(property "Reference" "#PWR0509"
 			(at 177.8 109.22 0)
 			(effects
@@
 			(project "table-zamboni"
 				(path "/6b8b7632-a6ae-4a95-9a82-5604ab03d2a7/e5c972da-9e3b-4905-a822-7ee0d7b899b3"
-					(reference "#PWR0512")
+					(reference "#PWR0509")
 					(unit 1)
 				)
@@
 		(dnp no)
 		(fields_autoplaced yes)
-		(property "Reference" "#PWR0504"
+		(property "Reference" "#PWR0505"
 			(at 78.74 59.69 0)
 			(effects
@@
 			(project "table-zamboni"
 				(path "/6b8b7632-a6ae-4a95-9a82-5604ab03d2a7/e5c972da-9e3b-4905-a822-7ee0d7b899b3"
-					(reference "#PWR0504")
+					(reference "#PWR0505")
 					(unit 1)
 				)
@@
 		(dnp no)
 		(fields_autoplaced yes)
-		(property "Reference" "R505"
+		(property "Reference" "R506"
 			(at 186.69 105.4099 0)
 			(effects
@@
 			(project "table-zamboni"
 				(path "/6b8b7632-a6ae-4a95-9a82-5604ab03d2a7/e5c972da-9e3b-4905-a822-7ee0d7b899b3"
-					(reference "R505")
+					(reference "R506")
 					(unit 1)
 				)
@@
 		(dnp no)
 		(fields_autoplaced yes)
-		(property "Reference" "#PWR0503"
+		(property "Reference" "#PWR0511"
 			(at 189.23 72.39 0)
 			(effects
@@
 			(project "table-zamboni"
 				(path "/6b8b7632-a6ae-4a95-9a82-5604ab03d2a7/e5c972da-9e3b-4905-a822-7ee0d7b899b3"
-					(reference "#PWR0503")
+					(reference "#PWR0511")
 					(unit 1)
 				)
@@
 		(on_board yes)
 		(dnp no)
-		(property "Reference" "Q501"
+		(property "Reference" "Q502"
 			(at 179.832 121.158 0)
 			(effects
@@
 			(project "table-zamboni"
 				(path "/6b8b7632-a6ae-4a95-9a82-5604ab03d2a7/e5c972da-9e3b-4905-a822-7ee0d7b899b3"
-					(reference "Q501")
+					(reference "Q502")
 					(unit 1)
 				)
@@
 		(dnp no)
 		(fields_autoplaced yes)
-		(property "Reference" "R504"
+		(property "Reference" "R502"
 			(at 67.31 116.8399 0)
 			(effects
@@
 			(project "table-zamboni"
 				(path "/6b8b7632-a6ae-4a95-9a82-5604ab03d2a7/e5c972da-9e3b-4905-a822-7ee0d7b899b3"
-					(reference "R504")
+					(reference "R502")
 					(unit 1)
 				)
@@
 		(dnp no)
 		(fields_autoplaced yes)
-		(property "Reference" "#PWR0520"
+		(property "Reference" "#PWR0521"
 			(at 250.19 121.92 0)
 			(effects
@@
 			(project "table-zamboni"
 				(path "/6b8b7632-a6ae-4a95-9a82-5604ab03d2a7/e5c972da-9e3b-4905-a822-7ee0d7b899b3"
-					(reference "#PWR0520")
+					(reference "#PWR0521")
 					(unit 1)
 				)
@@
 		(dnp no)
 		(fields_autoplaced yes)
-		(property "Reference" "#PWR0519"
+		(property "Reference" "#PWR0510"
 			(at 189.23 40.64 0)
 			(effects
@@
 			(project "table-zamboni"
 				(path "/6b8b7632-a6ae-4a95-9a82-5604ab03d2a7/e5c972da-9e3b-4905-a822-7ee0d7b899b3"
-					(reference "#PWR0519")
+					(reference "#PWR0510")
 					(unit 1)
 				)
@@
 		(on_board yes)
 		(dnp no)
-		(property "Reference" "Q502"
+		(property "Reference" "Q501"
 			(at 179.832 57.658 0)
 			(effects
@@
 			(project "table-zamboni"
 				(path "/6b8b7632-a6ae-4a95-9a82-5604ab03d2a7/e5c972da-9e3b-4905-a822-7ee0d7b899b3"
-					(reference "Q502")
+					(reference "Q501")
 					(unit 1)
 				)
@@
 		(dnp no)
 		(fields_autoplaced yes)
-		(property "Reference" "#PWR0511"
+		(property "Reference" "#PWR0503"
 			(at 64.77 92.71 0)
 			(effects
@@
 			(project "table-zamboni"
 				(path "/6b8b7632-a6ae-4a95-9a82-5604ab03d2a7/e5c972da-9e3b-4905-a822-7ee0d7b899b3"
-					(reference "#PWR0511")
+					(reference "#PWR0503")
 					(unit 1)
 				)
@@
 		(dnp no)
 		(fields_autoplaced yes)
-		(property "Reference" "#PWR0514"
+		(property "Reference" "#PWR0512"
 			(at 189.23 104.14 0)
 			(effects
@@
 			(project "table-zamboni"
 				(path "/6b8b7632-a6ae-4a95-9a82-5604ab03d2a7/e5c972da-9e3b-4905-a822-7ee0d7b899b3"
-					(reference "#PWR0514")
+					(reference "#PWR0512")
 					(unit 1)
 				)
@@
 		(dnp no)
 		(fields_autoplaced yes)
-		(property "Reference" "#PWR0521"
+		(property "Reference" "#PWR0508"
 			(at 177.8 45.72 0)
 			(effects
@@
 			(project "table-zamboni"
 				(path "/6b8b7632-a6ae-4a95-9a82-5604ab03d2a7/e5c972da-9e3b-4905-a822-7ee0d7b899b3"
-					(reference "#PWR0521")
+					(reference "#PWR0508")
 					(unit 1)
 				)
@@
 		(dnp no)
 		(fields_autoplaced yes)
-		(property "Reference" "#PWR0518"
+		(property "Reference" "#PWR0519"
 			(at 237.49 121.92 0)
 			(effects
@@
 			(project "table-zamboni"
 				(path "/6b8b7632-a6ae-4a95-9a82-5604ab03d2a7/e5c972da-9e3b-4905-a822-7ee0d7b899b3"
-					(reference "#PWR0518")
+					(reference "#PWR0519")
 					(unit 1)
 				)
@@
 		(dnp no)
 		(fields_autoplaced yes)
-		(property "Reference" "#PWR0510"
+		(property "Reference" "#PWR0520"
 			(at 250.19 58.42 0)
 			(effects
@@
 			(project "table-zamboni"
 				(path "/6b8b7632-a6ae-4a95-9a82-5604ab03d2a7/e5c972da-9e3b-4905-a822-7ee0d7b899b3"
-					(reference "#PWR0510")
+					(reference "#PWR0520")
 					(unit 1)
 				)
@@
 		(dnp no)
 		(fields_autoplaced yes)
-		(property "Reference" "#PWR0509"
+		(property "Reference" "#PWR0518"
 			(at 237.49 58.42 0)
 			(effects
@@
 			(project "table-zamboni"
 				(path "/6b8b7632-a6ae-4a95-9a82-5604ab03d2a7/e5c972da-9e3b-4905-a822-7ee0d7b899b3"
-					(reference "#PWR0509")
+					(reference "#PWR0518")
 					(unit 1)
 				)
@@
 		(dnp no)
 		(fields_autoplaced yes)
-		(property "Reference" "#PWR0508"
+		(property "Reference" "#PWR0516"
 			(at 222.25 40.64 0)
 			(effects
@@
 			(project "table-zamboni"
 				(path "/6b8b7632-a6ae-4a95-9a82-5604ab03d2a7/e5c972da-9e3b-4905-a822-7ee0d7b899b3"
-					(reference "#PWR0508")
+					(reference "#PWR0516")
 					(unit 1)
 				)
@@
 		(dnp no)
 		(fields_autoplaced yes)
-		(property "Reference" "#PWR0515"
+		(property "Reference" "#PWR0513"
 			(at 189.23 135.89 0)
 			(effects
@@
 			(project "table-zamboni"
 				(path "/6b8b7632-a6ae-4a95-9a82-5604ab03d2a7/e5c972da-9e3b-4905-a822-7ee0d7b899b3"
-					(reference "#PWR0515")
+					(reference "#PWR0513")
 					(unit 1)
 				)
@@
 		(dnp no)
 		(fields_autoplaced yes)
-		(property "Reference" "#PWR0505"
+		(property "Reference" "#PWR0514"
 			(at 217.17 83.82 0)
 			(effects
@@
 			(project "table-zamboni"
 				(path "/6b8b7632-a6ae-4a95-9a82-5604ab03d2a7/e5c972da-9e3b-4905-a822-7ee0d7b899b3"
-					(reference "#PWR0505")
+					(reference "#PWR0514")
 					(unit 1)
 				)
@@
 		(dnp no)
 		(fields_autoplaced yes)
-		(property "Reference" "#PWR0513"
+		(property "Reference" "#PWR0504"
 			(at 64.77 116.84 0)
 			(effects
@@
 			(project "table-zamboni"
 				(path "/6b8b7632-a6ae-4a95-9a82-5604ab03d2a7/e5c972da-9e3b-4905-a822-7ee0d7b899b3"
-					(reference "#PWR0513")
+					(reference "#PWR0504")
 					(unit 1)
 				)
@@
 		(dnp no)
 		(fields_autoplaced yes)
-		(property "Reference" "R507"
+		(property "Reference" "R503"
 			(at 175.26 46.9899 0)
 			(effects
@@
 			(project "table-zamboni"
 				(path "/6b8b7632-a6ae-4a95-9a82-5604ab03d2a7/e5c972da-9e3b-4905-a822-7ee0d7b899b3"
-					(reference "R507")
+					(reference "R503")
 					(unit 1)
 				)
@@
 		(dnp no)
 		(fields_autoplaced yes)
-		(property "Reference" "R501"
+		(property "Reference" "R505"
 			(at 186.69 41.9099 0)
 			(effects
@@
 			(project "table-zamboni"
 				(path "/6b8b7632-a6ae-4a95-9a82-5604ab03d2a7/e5c972da-9e3b-4905-a822-7ee0d7b899b3"
-					(reference "R501")
+					(reference "R505")
 					(unit 1)
 				)
@@
 		(dnp no)
 		(fields_autoplaced yes)
-		(property "Reference" "C505"
+		(property "Reference" "C504"
 			(at 233.68 109.2199 0)
 			(effects
@@
 			(project "table-zamboni"
 				(path "/6b8b7632-a6ae-4a95-9a82-5604ab03d2a7/e5c972da-9e3b-4905-a822-7ee0d7b899b3"
-					(reference "C505")
-					(unit 1)
-				)
+					(reference "C504")
+					(unit 1)
+				)
