File: Main_PCB/imu.kicad_sch (KiCad schematic)
At the start: 4 parts, among them U501 LSM6DS3

Commit message: First draft of schematic complete. Still need to verify it is correct before proceeding to pcb.
Parts:
- U401: renamed from U501; value LSM6DS3 -> LSM6DSO32X
- renumbered C506 to C401, C505 to C402, R505 to R401
Changed lines of the file:
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@@
 		(on_board yes)
 		(dnp no)
-		(property "Reference" "U501"
+		(property "Reference" "U401"
 			(at 131.826 93.218 0)
 			(effects
@@
 			)
 		)
-		(property "Value" "LSM6DS3"
+		(property "Value" "LSM6DSO32X"
 			(at 131.826 95.758 0)
 			(effects
@@
 			(project "table-zamboni"
 				(path "/6b8b7632-a6ae-4a95-9a82-5604ab03d2a7/8cce2de5-db49-4c04-aeca-96191d207de7"
-					(reference "U501")
+					(reference "U401")
 					(unit 1)
 				)
@@
 		(dnp no)
 		(fields_autoplaced yes)
-		(property "Reference" "C505"
+		(property "Reference" "C402"
 			(at 138.43 49.53 90)
 			(effects
@@
 			(project "table-zamboni"
 				(path "/6b8b7632-a6ae-4a95-9a82-5604ab03d2a7/8cce2de5-db49-4c04-aeca-96191d207de7"
-					(reference "C505")
+					(reference "C402")
 					(unit 1)
 				)
@@
 		(dnp no)
 		(fields_autoplaced yes)
-		(property "Reference" "#PWR0502"
+		(property "Reference" "#PWR0401"
 			(at 92.71 81.28 0)
 			(effects
@@
 			(project "table-zamboni"
 				(path "/6b8b7632-a6ae-4a95-9a82-5604ab03d2a7/8cce2de5-db49-4c04-aeca-96191d207de7"
-					(reference "#PWR0502")
+					(reference "#PWR0401")
 					(unit 1)
 				)
@@
 		(dnp no)
 		(fields_autoplaced yes)
-		(property "Reference" "#PWR0501"
+		(property "Reference" "#PWR0405"
 			(at 128.27 101.6 0)
 			(effects
@@
 			(project "table-zamboni"
 				(path "/6b8b7632-a6ae-4a95-9a82-5604ab03d2a7/8cce2de5-db49-4c04-aeca-96191d207de7"
-					(reference "#PWR0501")
+					(reference "#PWR0405")
 					(unit 1)
 				)
@@
 		(dnp no)
 		(fields_autoplaced yes)
-		(property "Reference" "#PWR0515"
+		(property "Reference" "#PWR0403"
 			(at 113.03 66.04 0)
 			(effects
@@
 			(project "table-zamboni"
 				(path "/6b8b7632-a6ae-4a95-9a82-5604ab03d2a7/8cce2de5-db49-4c04-aeca-96191d207de7"
-					(reference "#PWR0515")
+					(reference "#PWR0403")
 					(unit 1)
 				)
@@
 		(dnp no)
 		(fields_autoplaced yes)
-		(property "Reference" "#PWR0503"
+		(property "Reference" "#PWR0404"
 			(at 128.27 52.07 0)
 			(effects
@@
 			(project "table-zamboni"
 				(path "/6b8b7632-a6ae-4a95-9a82-5604ab03d2a7/8cce2de5-db49-4c04-aeca-96191d207de7"
-					(reference "#PWR0503")
+					(reference "#PWR0404")
 					(unit 1)
 				)
@@
 		(dnp no)
 		(fields_autoplaced yes)
-		(property "Reference" "#PWR0504"
+		(property "Reference" "#PWR0402"
 			(at 106.68 95.25 0)
 			(effects
@@
 			(project "table-zamboni"
 				(path "/6b8b7632-a6ae-4a95-9a82-5604ab03d2a7/8cce2de5-db49-4c04-aeca-96191d207de7"
-					(reference "#PWR0504")
+					(reference "#PWR0402")
 					(unit 1)
 				)
@@
 		(dnp no)
 		(fields_autoplaced yes)
-		(property "Reference" "#PWR0514"
+		(property "Reference" "#PWR0406"
 			(at 146.05 66.04 0)
 			(effects
@@
 			(project "table-zamboni"
 				(path "/6b8b7632-a6ae-4a95-9a82-5604ab03d2a7/8cce2de5-db49-4c04-aeca-96191d207de7"
-					(reference "#PWR0514")
+					(reference "#PWR0406")
 					(unit 1)
 				)
@@
 		(dnp no)
 		(fields_autoplaced yes)
-		(property "Reference" "R505"
+		(property "Reference" "R401"
 			(at 104.14 91.4399 0)
 			(effects
@@
 			(project "table-zamboni"
 				(path "/6b8b7632-a6ae-4a95-9a82-5604ab03d2a7/8cce2de5-db49-4c04-aeca-96191d207de7"
-					(reference "R505")
+					(reference "R401")
 					(unit 1)
 				)
@@
 		(dnp no)
 		(fields_autoplaced yes)
-		(property "Reference" "C506"
+		(property "Reference" "C401"
 			(at 120.65 49.53 90)
 			(effects
@@
 			(project "table-zamboni"
 				(path "/6b8b7632-a6ae-4a95-9a82-5604ab03d2a7/8cce2de5-db49-4c04-aeca-96191d207de7"
-					(reference "C506")
-					(unit 1)
-				)
+					(reference "C401")
+					(unit 1)
+				)

Commit message: Adding changes. Changes made to cleanup schematic before pcb layout.
Parts:
- renumbered C401 to C11, C402 to C12, R401 to R23, U401 to U5
Connections:
- net IMU_CS renamed CS
- net IMU_INT1 renamed INT1
- net SPI_MISO renamed MISO
- net SPI_MOSI renamed MOSI
- net SPI_SCK renamed SCK
Other:
- moved on the sheet: C11, C12, R23, U5
