File: Main_PCB/table-zamboni.kicad_sch (KiCad schematic)
At the start: 8 parts, among them J101 Conn_01x06, U302 ESP32-S3-WROOM-1

Commit message: First draft of schematic complete. Still need to verify it is correct before proceeding to pcb.
Parts:
- removed J101: Conn_01x06, symbol Connector_Generic:Conn_01x06
- removed R102: 22R, symbol Device:R
- added C101: 100nF, symbol Device:C
- added C102, C105: 10uF, symbol Device:C
- added C103, C104: 1uF, symbol Device:C
- added D102: LED, symbol Device:LED
- added J101: USB_B_Micro, symbol Connector:USB_B_Micro
- added J102: Conn_01x02, symbol Connector_Generic:Conn_01x02
- added Q101, Q102: SS8050, symbol Device:Q_NPN
- added R105, R108, R109: 10k, symbol Device:R
- added R106, R114: 1k, symbol Device:R
- added R110, R111, R115, R116: 0R, symbol Device:R
- added R112: 22.1k, symbol Device:R
- added R113: 47.5k, symbol Device:R
- added SW101, SW102: SW_Push, symbol Switch:SW_Push
- added U102: CP2102N-Axx-xQFN28, Package_DFN_QFN:QFN-28-1EP_5x5mm_P0.5mm_EP3.35x3.35mm, symbol Interface_USB:CP2102N-Axx-xQFN28
- added U103: USBLC6-2SC6, Package_TO_SOT_SMD:SOT-23-6, symbol Power_Protection:USBLC6-2SC6
- R101: value 22R -> 10k
- renumbered R103 to R102, R104 to R103, R105 to R104, R106 to R107, U302 to U101
Connections:
- net +3.3V: now also R101.1, C101.1, C102.1, C105.1, R105.1, R114.1, U102.6 (VDD), U102.7 (VREGIN)
- net EN: now also R101.2, C103.1, R110.2, SW102.2
- net GND: now also C101.2, C102.2, C103.2, C104.2, C105.2, D102.1 (K), J101.5 (GND), J101.6 (Shield), J102.2 (Pin_2), R113.2, SW101.1, SW102.1, U102.29 (GND), U102.3 (GND), U103.2 (GND)
- net IO0: now also R105.2, R111.2, SW101.2
- net LEFT_XSHUT: now also U101.18 (GPIO10/TOUCH10/ADC1_CH9/FSPICS0/FSPIIO4/SUBSPICS0)
- net RIGHT_XSHUT: now also U101.19 (GPIO11/TOUCH11/ADC2_CH0/FSPID/FSPIIO5/SUBSPID)
- net USB_D+: now also U102.4 (D+), U103.6 (I/O1); no longer R101.2
- net USB_D-: now also U102.5 (D-), U103.4 (I/O2)
- net at U101.14 (GPIO20/U1CTS/ADC2_CH9/CLK_OUT1/USB_D+): no longer R101.1
- net I2C_SDA: now reaches U101.12 (GPIO8/TOUCH8/ADC1_CH7/SUBSPICS1)
- net I2C_SCL: now reaches U101.17 (GPIO9/TOUCH9/ADC1_CH8/FSPIHD/SUBSPIHD)
- net MOTOR_ENABLE: now reaches U101.33 (MTDO/GPIO40/CLK_OUT2)
- net U0RXD: now reaches U101.36 (U0RXD/GPIO44/CLK_OUT2)
- net U0RXD: now also R115.1
- net U0TXD: now reaches U101.37 (U0TXD/GPIO43/CLK_OUT1)
- net U0TXD: now also R116.1
- net SWEEP_PWM renamed SERVO_CONTROL
- new net: J101.2 (D-), U103.3 (I/O2)
- new net: J101.3 (D+), U103.1 (I/O1)
- new net: R115.2, U102.26 (TXD)
- new net: R116.2, U102.25 (RXD)
- new net: Q102.B, R109.1
- new net: Q102.C, R111.1
- new net: D102.2 (A), R106.2
- new net: Q101.C, R110.1
- new net: Q101.B, R108.2
- new net: C104.1, R112.1, R113.1, U102.8 (VBUS)
- new net: R114.2, U102.9 (~{RST})
- new net +BATT: J102.1 (Pin_1)
- new net DTR: Q102.E, R108.1, U102.28 (~{DTR})
- new net RTS: Q101.E, R109.2, U102.24 (~{RTS})
- new net VBUS: J101.1 (VBUS), R106.1, R112.2, U103.5 (VBUS)
- no-connect marks 3 -> 20
Other:
- removed sheet ESP32
- added sheet ToF Sensors (tof_sensors.kicad_sch)
- sheet Motors ports: added SERVO_PWM, STBY; removed SWEEP_PWM
- note added: "Auto Program Truth Table"
- note added: "Auto Programming Circuit"
- note added: "B"
- note added: "BOOT"
- note added: "C"
- note added: "E"
- note added: "EN/RESET"
- note added: "Micro USB"
- note added: "USB to UART"
- note removed: "+5V_Battery"
- note removed: "+BATT"
- note removed: "3.3V"
- note removed: "5V"
- note removed: "BLOCK DIAGRAM"
- note removed: "GPIO-Left_Motor"
- note removed: "GPIO-Right_Motor"
- note removed: "GPIO-Servo"
- note removed: "GPIO0, GPIO3, GPIO45, GPIO46"
- note removed: "I2C"
- note removed: "Microcontroller: ESP32-S3 WROOM-1-N8"
- note removed: "SPI"
- note removed: "STRAPPING PINS:"
- note removed: "TABLE ZAMBONI DEVELOPMENT BOARD"
- note removed: "USB_DATA"
- note removed: "V_BUS"
- moved on the sheet: R102, R103, R104, R107, U101

Commit message: Added decoupling capacitors, pulldown resistors, test points, and more. Still need to finish verifying schematic before PCB layout.
Parts:
- removed J102: Conn_01x02, symbol Connector_Generic:Conn_01x02
- added R117: 220R, symbol Device:R
- added TP101: +BATT, symbol Connector:TestPoint
- added TP102: +5V_Battery, symbol Connector:TestPoint
- added TP103: VBUS, symbol Connector:TestPoint
- added TP104: +5V, symbol Connector:TestPoint
- added TP105: +3.3V, symbol Connector:TestPoint
- added TP106: +2.8V, symbol Connector:TestPoint
- added TP107: GND, symbol Connector:TestPoint
- added TP108: EN, symbol Connector:TestPoint
- added TP109: IO0, symbol Connector:TestPoint
- added TP110: UART_TX, symbol Connector:TestPoint
- added TP111: UART_RX, symbol Connector:TestPoint
- added TP112: I2C_SDA, symbol Connector:TestPoint
- added TP113: I2C_SCL, symbol Connector:TestPoint
- added TP114: IMU_CS, symbol Connector:TestPoint
- added TP115: IMU_SCLK, symbol Connector:TestPoint
- added TP116: PWR_STAT, symbol Connector:TestPoint
- added TP117: MTR_STBY, symbol Connector:TestPoint
- added TP118: LEFT_XSHUT, symbol Connector:TestPoint
- added TP119: RIGHT_XSHUT, symbol Connector:TestPoint
Connections:
- net +3.3V: now also TP105.1
- net +BATT: now also TP101.1
- net EN: now also TP108.1
- net GND: now also TP107.1
- net I2C_SCL: now also TP113.1
- net I2C_SDA: now also TP112.1
- net IMU_CS: now also TP114.1
- net IMU_SPI_SCK: now also TP115.1
- net IO0: now also TP109.1
- net LEFT_XSHUT: now also TP118.1
- net MOTOR_ENABLE: now also TP117.1
- net POWER_STATUS: now also TP116.1
- net RIGHT_XSHUT: now also TP119.1
- net SERVO_CONTROL: now also R117.1; no longer U101.35 (MTMS/GPIO42)
- net U0RXD: now also TP111.1
- net U0TXD: now also TP110.1
- net VBUS: now also TP103.1
- new net: R117.2, U101.35 (MTMS/GPIO42)
- new net +2V8: TP106.1
- new net +5V: TP104.1
- new net +5V_Battery: TP102.1
Other:
- sheet ToF Sensors ports: added TOF_LEFT_DISABLE, TOF_RIGHT_DISABLE; removed TOF_LEFT_XSHUT, TOF_RIGHT_XSHUT
- note added: "Test Points"

Commit message: Adding changes. Changes made to cleanup schematic before pcb layout.
Parts:
- removed C104: 1uF, symbol Device:C
- removed C105: 10uF, symbol Device:C
- removed D102: LED, symbol Device:LED
- removed J101: USB_B_Micro, symbol Connector:USB_B_Micro
- removed Q101, Q102: SS8050, symbol Device:Q_NPN
- removed R102, R103, R104, R107, R117: 220R, symbol Device:R
- removed R106, R114: 1k, symbol Device:R
- removed R108, R109: 10k, symbol Device:R
- removed R110, R111, R115, R116: 0R, symbol Device:R
- removed R112: 22.1k, symbol Device:R
- removed R113: 47.5k, symbol Device:R
- removed TP101: +BATT, symbol Connector:TestPoint
- removed TP102: +5V_Battery, symbol Connector:TestPoint
- removed TP103: VBUS, symbol Connector:TestPoint
- removed TP104: +5V, symbol Connector:TestPoint
- removed TP105: +3.3V, symbol Connector:TestPoint
- removed TP106: +2.8V, symbol Connector:TestPoint
- removed TP107: GND, symbol Connector:TestPoint
- removed TP108: EN, symbol Connector:TestPoint
- removed TP109: IO0, symbol Connector:TestPoint
- removed TP110: UART_TX, symbol Connector:TestPoint
- removed TP111: UART_RX, symbol Connector:TestPoint
- removed TP112: I2C_SDA, symbol Connector:TestPoint
- removed TP113: I2C_SCL, symbol Connector:TestPoint
- removed TP114: IMU_CS, symbol Connector:TestPoint
- removed TP115: IMU_SCLK, symbol Connector:TestPoint
- removed TP116: PWR_STAT, symbol Connector:TestPoint
- removed TP117: MTR_STBY, symbol Connector:TestPoint
- removed TP118: LEFT_XSHUT, symbol Connector:TestPoint
- removed TP119: RIGHT_XSHUT, symbol Connector:TestPoint
- removed U101: ESP32-S3-WROOM-1, PCM_Espressif:ESP32-S3-WROOM-1, symbol PCM_Espressif:ESP32-S3-WROOM-1
- removed U102: CP2102N-Axx-xQFN28, Package_DFN_QFN:QFN-28-1EP_5x5mm_P0.5mm_EP3.35x3.35mm, symbol Interface_USB:CP2102N-Axx-xQFN28
- removed U103: USBLC6-2SC6, Package_TO_SOT_SMD:SOT-23-6, symbol Power_Protection:USBLC6-2SC6
- added C28: 0.1uF, symbol Device:C
- added D3: 3.3V_MCU, symbol Device:LED
- added D7: CDSOD323-T03, symbol Device:D_Zener
- added J1, J2: Conn_01x04, symbol Connector_Generic:Conn_01x04
- added J9: Conn_01x06, symbol Connector_Generic:Conn_01x06
- added R2, R3: 100Ω, symbol Device:R
- added R27: 65Ω, symbol Device:R
- added R35, R36, R37, R38: 220Ω, symbol Device:R
- added U1: DESD3V3S2UTQ-7, symbol desd3v3s2utq-7:DESD3V3S2UTQ-7
- added U9: ESP32-S3-WROOM-1(N8), symbol esp32_s3:ESP32-S3-WROOM-1(N8)
- renumbered C101 to C1, C102 to C2, C103 to C3, R101 to R1, R105 to R5, SW101 to SW1, SW102 to SW2
Connections:
- net +3.3V: now also C28.1, D7.1 (K), J2.1 (Pin_1), R27.1, U9.2 (3V3)
- net ENCODER_LEFT_A: now also R38.2
- net ENCODER_LEFT_B: now also R37.1
- net ENCODER_RIGHT_A: now also R36.1
- net ENCODER_RIGHT_B: now also R35.1
- net GND: now also C28.2, D3.1 (K), D7.2 (A), J1.4 (Pin_4), J2.4 (Pin_4), U1.3 (GND), U9.1 (GND), U9.40 (GND), U9.41 (EPAD)
- net I2C_SCL: now also U9.12 (IO8)
- net I2C_SDA: now also U9.17 (IO9)
- net IMU_CS: now also U9.13 (IO19)
- net IMU_INT1: now also U9.14 (IO20)
- net IMU_SPI_MISO: now also U9.21 (IO13)
- net IMU_SPI_MOSI: now also U9.19 (IO11)
- net IMU_SPI_SCK: now also U9.20 (IO12)
- net LEFT_MTR_IN1: now also U9.22 (IO14)
- net LEFT_MTR_IN2: now also U9.23 (IO21)
- net LEFT_XSHUT: now also U9.9 (IO16)
- net MOTOR_ENABLE: now also U9.33 (IO40)
- net RIGHT_MTR_IN1: now also U9.24 (IO47)
- net RIGHT_MTR_IN2: now also U9.25 (IO48)
- net RIGHT_XSHUT: now also U9.10 (IO17)
- net U0RXD: now also U9.36 (RXD0)
- net U0TXD: now also U9.37 (TXD0)
- net EN renamed ESP_EN
- net ESP_EN: now also U9.3 (EN)
- net IO0 renamed ESP_IO0
- net ESP_IO0: now also U9.27 (IO0)
- new net: R38.1, U9.28 (IO35)
- new net: R37.2, U9.29 (IO36)
- new net: R36.2, U9.30 (IO37)
- new net: R35.2, U9.31 (IO38)
- new net: R3.2, U9.6 (IO6)
- new net: R2.2, U9.7 (IO7)
- new net: D3.2 (A), R27.2
- new net ECHO: J2.3 (Pin_3), R2.1, U1.2 (SIG2)
- new net START_BUTTON: U9.35 (IO42)
- new net START_LED: U9.34 (IO41)
- new net TRIG: J2.2 (Pin_2), R3.1, U1.1 (SIG1)
- new net V_MOTOR: J1.1 (Pin_1)
- new net ~{MOTOR_FAULT}: U9.32 (IO39)
- no-connect marks 20 -> 3
Other:
- added sheet USB to UART (usb_to_uart.kicad_sch)
- sheet IMU ports: added CS, INT1, MISO, MOSI, SCK; removed IMU_CS, IMU_INT1, SPI_MISO, SPI_MOSI, SPI_SCK
- sheet Motors ports: added ~{FAULT}, ~{SLEEP}; removed PWMA, PWMB, SERVO_PWM, STBY
- sheet Power Management ports: added none; removed PWR_STAT
- sheet ToF Sensors: file tof_sensors.kicad_sch -> tof.kicad_sch
- note added: "Button & LED Breakout Board Connection"
- note added: "LED resistor value calculation: Ohm's Law: V=IR -> R=V/I V_{S} = 3.3V (supply voltage) V_{F} = 2.1V (LED forward voltage) I = 20mA R= (V_{S} - V_{F})/I R = (3.3V - 2.1V)/ (20mA) = 60 Ω ∴ choose R = 65 Ω"
- note added: "Status LED (3.3V)"
- note added: "ToF Breakout Board Connection"
- note added: "Ultrasonic Distance Sensor Connection (with ESD protection)"
- note removed: "Auto Program Truth Table"
- note removed: "Auto Programming Circuit"
- note removed: "B"
- note removed: "C"
- note removed: "E"
- note removed: "Micro USB"
- note removed: "Test Points"
- note removed: "USB to UART"
- moved on the sheet: C1, C2, C3, R1, R5, SW1, SW2
