File: ToF_PCB/tof_sensors.kicad_sch (KiCad schematic)
At the start: 22 parts, among them J1 Conn_01x06, Q1 2N7002, Q2 2N7002, U1 LP5907MFX-2.8, U2 VL53L4CD, U3 VL53L4CD

Commit message: Updated pcb layout. Moved ToF sensors to back of board.
Parts:
- added C7: 100nF, Capacitor_SMD:C_0201_0603Metric, symbol Device:C
- added U4: USBLC6-4SC6, Package_TO_SOT_SMD:SOT-23-6, symbol Power_Protection:USBLC6-4SC6
- C1: footprint Capacitor_SMD:C_0805_2012Metric_Pad1.18x1.45mm_HandSolder -> Capacitor_SMD:C_0504_1310Metric
- J1: footprint Connector_JST:JST_SH_SM06B-SRSS-TB_1x06-1MP_P1.00mm_Horizontal -> Connector_JST:JST_SH_BM06B-SRSS-TB_1x06-1MP_P1.00mm_Vertical
Connections:
- net +3.3V: now also J1.6 (Pin_6), C7.1, U4.5 (VBUS); no longer J1.1 (Pin_1)
- net GND: now also J1.1 (Pin_1), C7.2, U4.2 (GND); no longer J1.6 (Pin_6)
- net SCL: now also U4.6 (I/O4)
- net SDA: now also U4.1 (I/O1)
- net TOF_LEFT_DISABLE: now also J1.5 (Pin_5), U4.4 (I/O3); no longer J1.2 (Pin_2)
- net TOF_RIGHT_DISABLE: now also J1.2 (Pin_2), U4.3 (I/O2); no longer J1.5 (Pin_5)
- net RIGHT_XSHUT: now reaches Q2.3 (D), R4.2, U3.5 (XSHUT)
- net LEFT_XSHUT: now reaches Q1.3 (D), R1.2, U2.5 (XSHUT)
